File: RAMPS1.4/RAMPS_1-41.brd (EAGLE design)
At the start: 101.6 x 60.9 mm, 88 parts, among them Q1 STP55NF06L, Q2 STP55NF06L, Q3 STP55NF06L, U1 ARDUINO_MEGA_SHIELD, X4 MSTBA4

Commit message: add libs
Parts:
- JP2, JP3, JP4, JP5, JP6: device pinhead:2X03 -> eagle-ramps:2X03
- R10: device adafruit:R0805 -> adafruit:R1206W
- U$4: device RepRapjr:A4988BREAKOUT -> e0:A4988BREAKOUT
- U$6: device RepRapjr:A4988BREAKOUT -> x:A4988BREAKOUT
- U1: device RepRapjr:ARDUINO_MEGA_SHIELD -> RepRapjr_o:ARDUINO_MEGA_SHIELD
- moved R16 10.2 mm to (38.1, 51.4), flipped to the bottom, turned to 0 degrees
- moved R19 9.96 mm to (55.2, 14.9), flipped to the bottom, turned to 90 degrees
- moved R18 6.74 mm to (29.5, 18.1), flipped to the bottom, turned to 90 degrees
- moved R17 5.83 mm to (53.0, 41.0), flipped to the bottom, turned to 0 degrees
- moved R10 5.21 mm to (78.7, 27.6), flipped to the bottom, turned to 0 degrees
- moved R8 5.08 mm to (59.6, 26.3), flipped to the bottom, turned to 90 degrees
- moved R20 2.31 mm to (72.7, 23.5), flipped to the bottom, turned to 270 degrees
- moved R2 0.65 mm to (33.2, 60.3)
- moved R6 0.64 mm to (40.3, 46.0)
- moved D1 0.32 mm to (50.6, 23.3)
Routing:
- net GND: track 668.0 -> 618.1 mm
- net E0-EN: track 87.9 -> 74.4 mm
- net VCC: track 352.8 -> 342.3 mm, vias 3 -> 2
- net D1: track 83.9 -> 76.2 mm
- net D2: track 86.5 -> 80.3 mm
- net D12: track 113.6 -> 107.5 mm
- net Y-EN: track 12.4 -> 6.73 mm
- net X-EN: track 81.0 -> 84.7 mm
- net +12V: track 230.1 -> 227.4 mm
- net D11: track 82.4 -> 80.2 mm
- net D4: track 72.5 -> 71.2 mm
- net X-STEP: track 4.76 -> 5.98 mm
- net Z-EN: track 6.09 -> 5.01 mm
- net N$40: track 13.3 -> 12.2 mm
- net D6: track 61.2 -> 60.3 mm
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Other:
- board size 101.6 x 60.9 mm -> 102.9 x 62.2 mm

Commit message: 160522
Parts:
- removed U$10: M05X2, RepRapjr:2X5
- removed U$5, U$7, U$8: A4988BREAKOUT, RepRapjr:A4988BREAKOUT
- removed U$9: M18_, SparkFun:1X18
- added AUX2: M05X2, RepRapjr_o:2X5
- added AUX4: M18_, SparkFun:1X18
- added J: (no value), rcl:R1206W
- added U$5E1: A4988BREAKOUT, e1:A4988BREAKOUT
- added U$7Y: A4988BREAKOUT, y:A4988BREAKOUT
- added Z: A4988BREAKOUT, z:A4988BREAKOUT
- R21, R22: device adafruit:R0805 -> adafruit:R0603
- moved R22 19.7 mm to (89.2, 66.7), flipped to the bottom, turned to 180 degrees
- moved R11 19.6 mm to (89.5, 40.8), flipped to the bottom, turned to 0 degrees
- moved R1 13.9 mm to (84.1, 41.1), flipped to the bottom, turned to 0 degrees
- moved R21 13.8 mm to (91.4, 65.9), flipped to the bottom, turned to 90 degrees
- moved R7 7.98 mm to (78.7, 41.0), flipped to the bottom, turned to 0 degrees
- moved R3 3.60 mm to (59.8, 47.7), turned to 180 degrees
- moved R5 1.06 mm to (39.7, 24.6)
- moved D1 0.97 mm to (49.6, 23.1)
- moved R20 0.71 mm to (73.3, 23.2), turned to 0 degrees
- moved JP4 0.71 mm to (43.8, 28.3)
- moved R8 0.64 mm to (59.6, 25.7)
- moved R19 0.50 mm to (55.7, 14.8)
- moved C4 0.48 mm to (55.2, 50.3)
- moved C3 0.32 mm to (34.0, 50.8)
- moved JP6 0.32 mm to (85.1, 28.3)
- renumbered U$3 to AUX3, U$4 to U$4E0, U$6 to U$6X
Connections:
- new net N$2: J.1, U1.D38
- net +12V: now also U$5E1.VMOT, U$7Y.VMOT, Z.VMOT; no longer U$5.VMOT, U$7.VMOT, U$8.VMOT
- net A10: now also AUX2.5; no longer U$10.5
- net A11: now also AUX2.10; no longer U$10.10
- net A12: now also AUX2.9; no longer U$10.9
- net A5: now also AUX2.3; no longer U$10.3
- net A9: now also AUX2.4; no longer U$10.4
- net D16: now also AUX4.18; no longer U$9.18
- net D17: now also AUX4.17; no longer U$9.17
- net D23: now also AUX4.16; no longer U$9.16
- net D25: now also AUX4.15; no longer U$9.15
- net D27: now also AUX4.14; no longer U$9.14
- net D29: now also AUX4.13; no longer U$9.13
- net D31: now also AUX4.12; no longer U$9.12
- net D32: now also AUX4.3; no longer U$9.3
- net D33: now also AUX4.11; no longer U$9.11
- net D35: now also AUX4.10; no longer U$9.10
- net D37: now also AUX4.9; no longer U$9.9
- net D39: now also AUX4.8; no longer U$9.8
- net D40: now also AUX2.6; no longer U$10.6
- net D41: now also AUX4.7; no longer U$9.7
- net D42: now also AUX2.8; no longer U$10.8
- net D43: now also AUX4.6; no longer U$9.6
- net D44: now also AUX2.7; no longer U$10.7
- net D45: now also AUX4.5; no longer U$9.5
- net D47: now also AUX4.4; no longer U$9.4
- net E1-DIR: now also U$5E1.DIR; no longer U$5.DIR
- net E1-EN: now also U$5E1.EN; no longer U$5.EN
- net E1-STEP: now also U$5E1.STEP; no longer U$5.STEP
- net GND: now also AUX2.2, AUX4.2, U$5E1.GND, U$5E1.GND@0, U$7Y.GND, U$7Y.GND@0, Z.GND, Z.GND@0; no longer U$10.2, U$5.GND, U$5.GND@0, U$7.GND, U$7.GND@0, U$8.GND, U$8.GND@0, U$9.2
- net N$12: now also U$5E1.2B; no longer U$5.2B
- net N$13: now also U$5E1.2A; no longer U$5.2A
- net N$16: now also U$5E1.1A; no longer U$5.1A
- net N$17: now also U$7Y.MS2; no longer U$7.MS2
- net N$18: now also U$5E1.1B; no longer U$5.1B
- net N$23: now also U$7Y.RST, U$7Y.SLP; no longer U$7.RST, U$7.SLP
- net N$24: now also U$5E1.RST, U$5E1.SLP; no longer U$5.RST, U$5.SLP
- net N$25: now also U$5E1.MS1; no longer U$5.MS1
- net N$28: now also U$7Y.2B; no longer U$7.2B
- net N$29: now also U$7Y.2A; no longer U$7.2A
- net N$30: now also U$7Y.1A; no longer U$7.1A
- net N$31: now also U$7Y.MS3; no longer U$7.MS3
- net N$33: now also U$7Y.MS1; no longer U$7.MS1
- net N$34: now also U$5E1.MS3; no longer U$5.MS3
- net N$35: now also U$5E1.MS2; no longer U$5.MS2
- net N$36: now also U$7Y.1B; no longer U$7.1B
- net N$37: now also Z.MS2; no longer U$8.MS2
- net N$38: now also Z.RST, Z.SLP; no longer U$8.RST, U$8.SLP
- net N$39: now also Z.MS3; no longer U$8.MS3
- net N$40: now also Z.MS1; no longer U$8.MS1
- net N$41: now also Z.2B; no longer U$8.2B
- net N$42: now also Z.2A; no longer U$8.2A
- net N$43: now also Z.1A; no longer U$8.1A
- net N$44: now also Z.1B; no longer U$8.1B
- net VCC: now also AUX2.1, AUX4.1, U$5E1.VDD, U$7Y.VDD, Z.VDD; no longer U$10.1, U$5.VDD, U$7.VDD, U$8.VDD, U$9.1
- net X-EN: now also J.2; no longer U1.D38
- net Y-DIR: now also U$7Y.DIR; no longer U$7.DIR
- net Y-EN: now also U$7Y.EN; no longer U$7.EN
- net Y-STEP: now also U$7Y.STEP; no longer U$7.STEP
- net Z-DIR: now also Z.DIR; no longer U$8.DIR
- net Z-EN: now also Z.EN; no longer U$8.EN
- net Z-STEP: now also Z.STEP; no longer U$8.STEP
Routing:
- net X-EN: track 84.7 -> 7.11 mm
- net N$2: track 0.00 -> 74.0 mm
- net SCL: track 23.5 -> 6.05 mm
- net THERM2: track 56.5 -> 40.1 mm
- net GND: track 618.1 -> 634.1 mm
- net THERM1: track 59.3 -> 45.1 mm
- net THERM0: track 57.1 -> 49.4 mm
- net D17: track 32.9 -> 26.2 mm
- net SDA: track 17.0 -> 12.3 mm
- net VCC: track 342.3 -> 338.9 mm
- net N$33: track 12.8 -> 9.77 mm
- net N$25: track 13.4 -> 10.6 mm
- net D32: track 26.7 -> 29.5 mm
- net E1-DIR: track 29.6 -> 26.9 mm
- net D4: track 71.2 -> 68.7 mm
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Other:
- board size 102.9 x 62.2 mm -> 102.9 x 61.9 mm
- board text added: "Endstops"
- board text added: "RAMPS1.4"
