File: RAMPS1.4/RAMPS_1-41.sch (EAGLE design)
At the start: 88 parts, among them Q1 STP55NF06L, Q2 STP55NF06L, Q3 STP55NF06L, U1 ARDUINO_MEGA_SHIELD, X4 MSTBA4

Commit message: add libs
Parts:
- JP2, JP3, JP4, JP5, JP6: device pinhead:PINHD-2X3 -> eagle-ramps:PINHD-2X3
- R10: device adafruit:R-US_R0805 -> adafruit:R-US_R1206W
- U$4: device RepRapjr:A4988BREAKOUT -> e0:A4988BREAKOUT
- U$6: device RepRapjr:A4988BREAKOUT -> x:A4988BREAKOUT
- U1: device RepRapjr:ARDUINO_MEGA_SHIELD -> RepRapjr_o:ARDUINO_MEGA_SHIELD
Changed lines of the file:
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@@
 <setting verticaltext="up"/>
 </settings>
-<grid distance="0.1" unitdist="inch" unit="inch" style="lines" multiple="1" display="no" altdistance="0.01" altunitdist="inch" altunit="inch"/>
+<grid distance="0.1" unitdist="inch" unit="inch" style="lines" multiple="1" display="yes" altdistance="0.01" altunitdist="inch" altunit="inch"/>
 <layers>
 <layer number="1" name="Top" color="4" fill="1" visible="no" active="no"/>
@@
 <layer number="17" name="Pads" color="2" fill="1" visible="no" active="no"/>
 <layer number="18" name="Vias" color="2" fill="1" visible="no" active="no"/>
-<layer number="19" name="Unrouted" color="13" fill="1" visible="no" active="no"/>
+<layer number="19" name="Unrouted" color="14" fill="1" visible="no" active="no"/>
 <layer number="20" name="Dimension" color="15" fill="1" visible="no" active="no"/>
 <layer number="21" name="tPlace" color="7" fill="1" visible="no" active="no"/>
@@
 <layer number="107" name="Crop" color="7" fill="1" visible="yes" active="yes"/>
 <layer number="108" name="Title" color="15" fill="1" visible="yes" active="yes"/>
+<layer number="114" name="114" color="7" fill="1" visible="yes" active="yes"/>
+<layer number="115" name="115" color="7" fill="1" visible="yes" active="yes"/>
 <layer number="116" name="Patch_BOT" color="9" fill="4" visible="yes" active="yes"/>
+<layer number="117" name="117" color="7" fill="1" visible="yes" active="yes"/>
+<layer number="119" name="119" color="7" fill="1" visible="yes" active="yes"/>
+<layer number="120" name="120" color="7" fill="1" visible="yes" active="yes"/>
 <layer number="121" name="_tsilk" color="7" fill="1" visible="yes" active="yes"/>
 <layer number="122" name="_bsilk" color="7" fill="1" visible="yes" active="yes"/>
 <layer number="125" name="_tNames" color="7" fill="1" visible="yes" active="yes"/>
+<layer number="129" name="129" color="7" fill="1" visible="yes" active="yes"/>
+<layer number="130" name="130" color="7" fill="1" visible="yes" active="yes"/>
+<layer number="133" name="133" color="7" fill="1" visible="yes" active="yes"/>
 <layer number="144" name="Drill_legend" color="7" fill="1" visible="yes" active="yes"/>
 <layer number="151" name="HeatSink" color="7" fill="1" visible="yes" active="yes"/>
@@
 <part name="R9" library="adafruit" deviceset="R-US_" device="R0805" value="100k"/>
 <part name="D1" library="diode" deviceset="1N4004" device=""/>
-<part name="U1" library="RepRapjr" deviceset="ARDUINO_MEGA_SHIELD" device=""/>
+<part name="U1" library="RepRapjr_o" deviceset="ARDUINO_MEGA_SHIELD" device=""/>
 <part name="LED1" library="led" deviceset="LED" device="CHIP-LED0805"/>
 <part name="GND2" library="supply1" deviceset="GND" device=""/>
@@
 <part name="GND19" library="supply1" deviceset="GND" device=""/>
 <part name="R6" library="adafruit" deviceset="R-US_" device="R0805" value="100k"/>
-<part name="JP2" library="pinhead" deviceset="PINHD-2X3" device=""/>
-<part name="JP3" library="pinhead" deviceset="PINHD-2X3" device=""/>
-<part name="JP5" library="pinhead" deviceset="PINHD-2X3" device=""/>
-<part name="JP4" library="pinhead" deviceset="PINHD-2X3" device=""/>
+<part name="JP2" library="eagle-ramps" deviceset="PINHD-2X3" device=""/>
+<part name="JP3" library="eagle-ramps" deviceset="PINHD-2X3" device=""/>
+<part name="JP5" library="eagle-ramps" deviceset="PINHD-2X3" device=""/>
+<part name="JP4" library="eagle-ramps" deviceset="PINHD-2X3" device=""/>
 <part name="R3" library="adafruit" deviceset="R-US_" device="R0805" value="100k"/>
 <part name="R5" library="adafruit" deviceset="R-US_" device="R0805" value="100k"/>
@@
 <part name="P+22" library="supply1" deviceset="+12V" device=""/>
 <part name="GND20" library="supply1" deviceset="GND" device=""/>
-<part name="JP6" library="pinhead" deviceset="PINHD-2X3" device=""/>
-<part name="R10" library="adafruit" deviceset="R-US_" device="R0805" value="100k"/>
+<part name="JP6" library="eagle-ramps" deviceset="PINHD-2X3" device=""/>
+<part name="R10" library="adafruit" deviceset="R-US_" device="R1206W" value="100k"/>
 <part name="Z-MOT" library="RepRapjr" deviceset="PINHD-1X4" device=""/>
 <part name="P+23" library="supply1" deviceset="VCC" device=""/>
@@
 <part name="GND31" library="supply1" deviceset="GND" device=""/>
 <part name="P+34" library="supply1" deviceset="+12V" device=""/>
-<part name="U$4" library="RepRapjr" deviceset="A4988BREAKOUT" device=""/>
+<part name="U$4" library="e0" deviceset="A4988BREAKOUT" device=""/>
 <part name="U$5" library="RepRapjr" deviceset="A4988BREAKOUT" device=""/>
-<part name="U$6" library="RepRapjr" deviceset="A4988BREAKOUT" device=""/>
+<part name="U$6" library="x" deviceset="A4988BREAKOUT" device=""/>
 <part name="U$7" library="RepRapjr" deviceset="A4988BREAKOUT" device=""/>
 <part name="U$8" library="RepRapjr" deviceset="A4988BREAKOUT" device=""/>

Commit message: 160522
Parts:
- removed U$10: M05X2, RepRapjr:M05X2
- removed U$3: M04X2, SparkFun:M04X2
- removed U$5, U$7, U$8: A4988BREAKOUT, RepRapjr:A4988BREAKOUT
- removed U$9: M18_, SparkFun:M18_
- added AUX2: M05X2, RepRapjr_o:M05X2
- added AUX3: M04X2, SparkFun:M04X2
- added AUX4: M18_, SparkFun:M18_
- added J: (no value), rcl:R-EU_R1206W
- added U$5E1: A4988BREAKOUT, e1:A4988BREAKOUT
- added U$7Y: A4988BREAKOUT, y:A4988BREAKOUT
- added Z: A4988BREAKOUT, z:A4988BREAKOUT
- R21, R22: device adafruit:R-US_R0805 -> adafruit:R-US_R0603
- renumbered U$4 to U$4E0, U$6 to U$6X
Connections:
- new net N$2: J.1, U1.D38
- net +12V: now also U$5E1.VMOT, U$7Y.VMOT, Z.VMOT; no longer U$5.VMOT, U$7.VMOT, U$8.VMOT
- net A10: now also AUX2.5; no longer U$10.5
- net A11: now also AUX2.10; no longer U$10.10
- net A12: now also AUX2.9; no longer U$10.9
- net A5: now also AUX2.3; no longer U$10.3
- net A9: now also AUX2.4; no longer U$10.4
- net D16: now also AUX4.18; no longer U$9.18
- net D17: now also AUX4.17; no longer U$9.17
- net D23: now also AUX4.16; no longer U$9.16
- net D25: now also AUX4.15; no longer U$9.15
- net D27: now also AUX4.14; no longer U$9.14
- net D29: now also AUX4.13; no longer U$9.13
- net D31: now also AUX4.12; no longer U$9.12
- net D32: now also AUX4.3; no longer U$9.3
- net D33: now also AUX4.11; no longer U$9.11
- net D35: now also AUX4.10; no longer U$9.10
- net D37: now also AUX4.9; no longer U$9.9
- net D39: now also AUX4.8; no longer U$9.8
- net D40: now also AUX2.6; no longer U$10.6
- net D41: now also AUX4.7; no longer U$9.7
- net D42: now also AUX2.8; no longer U$10.8
- net D43: now also AUX4.6; no longer U$9.6
- net D44: now also AUX2.7; no longer U$10.7
- net D45: now also AUX4.5; no longer U$9.5
- net D47: now also AUX4.4; no longer U$9.4
- net D49: now also AUX3.2; no longer U$3.2
- net D53: now also AUX3.6; no longer U$3.6
- net E1-DIR: now also U$5E1.DIR; no longer U$5.DIR
- net E1-EN: now also U$5E1.EN; no longer U$5.EN
- net E1-STEP: now also U$5E1.STEP; no longer U$5.STEP
- net GND: now also AUX2.2, AUX3.7, AUX4.2, U$5E1.GND@0, U$5E1.GND@1, U$7Y.GND@0, U$7Y.GND@1, Z.GND@0, Z.GND@1; no longer U$10.2, U$3.7, U$5.GND@0, U$5.GND@1, U$7.GND@0, U$7.GND@1, U$8.GND@0, U$8.GND@1, U$9.2
- net MISO: now also AUX3.3; no longer U$3.3
- net MOSI: now also AUX3.4; no longer U$3.4
- net N$12: now also U$5E1.2B; no longer U$5.2B
- net N$13: now also U$5E1.2A; no longer U$5.2A
- net N$16: now also U$5E1.1A; no longer U$5.1A
- net N$17: now also U$7Y.MS2; no longer U$7.MS2
- net N$18: now also U$5E1.1B; no longer U$5.1B
- net N$23: now also U$7Y.RST, U$7Y.SLEEP; no longer U$7.RST, U$7.SLEEP
- net N$24: now also U$5E1.RST, U$5E1.SLEEP; no longer U$5.RST, U$5.SLEEP
- net N$25: now also U$5E1.MS1; no longer U$5.MS1
- net N$28: now also U$7Y.2B; no longer U$7.2B
- net N$29: now also U$7Y.2A; no longer U$7.2A
- net N$30: now also U$7Y.1A; no longer U$7.1A
- net N$31: now also U$7Y.MS3; no longer U$7.MS3
- net N$33: now also U$7Y.MS1; no longer U$7.MS1
- net N$34: now also U$5E1.MS3; no longer U$5.MS3
- net N$35: now also U$5E1.MS2; no longer U$5.MS2
- net N$36: now also U$7Y.1B; no longer U$7.1B
- net N$37: now also Z.MS2; no longer U$8.MS2
- net N$38: now also Z.RST, Z.SLEEP; no longer U$8.RST, U$8.SLEEP
- net N$39: now also Z.MS3; no longer U$8.MS3
- net N$40: now also Z.MS1; no longer U$8.MS1
- net N$41: now also Z.2B; no longer U$8.2B
- net N$42: now also Z.2A; no longer U$8.2A
- net N$43: now also Z.1A; no longer U$8.1A
- net N$44: now also Z.1B; no longer U$8.1B
- net SCK: now also AUX3.5; no longer U$3.5
- net VCC: now also AUX2.1, AUX3.1, AUX4.1, U$5E1.VDD, U$7Y.VDD, Z.VDD; no longer U$10.1, U$3.1, U$5.VDD, U$7.VDD, U$8.VDD, U$9.1
- net X-EN: now also J.2; no longer U1.D38
- net Y-DIR: now also U$7Y.DIR; no longer U$7.DIR
- net Y-EN: now also U$7Y.EN; no longer U$7.EN
- net Y-STEP: now also U$7Y.STEP; no longer U$7.STEP
- net Z-DIR: now also Z.DIR; no longer U$8.DIR
- net Z-EN: now also Z.EN; no longer U$8.EN
- net Z-STEP: now also Z.STEP; no longer U$8.STEP
Other:
- note added: "-"
- note added: "BTN_ENC"
- note added: "BUZZ"
- note added: "CNT_RST"
- note added: "ENC1"
- note added: "ENC3"
- note added: "GND"
- note added: "LCD_CS"
- note added: "LCD_RST"
- note added: "LCD_SCK"
- note added: "LCD_SDA"
- note added: "RST_BUT"
- note added: "SD_CLK"
- note added: "SD_CS"
- note added: "SD_DIN"
- note added: "SD_R_CD"
- note added: "SD_R_DOUT"
- note added: "VCC"
